File: Schem/Z80HomeBrew/Z80HomeBrew.kicad_pcb (KiCad board)
At the start: 4 copper layers, 228.6 x 190.5 mm, 184 parts, among them IC1 Z80CTC, IC2 Z80SIO, IC3 Z80SIO, J1 PJ-037A, J10 RCJ-32265, J11 Conn_01x02_Pin, J12 Conn_01x02_Pin, J13 Conn_01x03, J14 Conn_01x04, J15 Conn_01x04, J16 Conn_01x04, J2 MSD-1-A, J3 0480370001, J4 0480370001, J5 0480370001, J6 STX-3120-3B, J7 Z80HomeBrewUser, J8 Conn_01x02_Pin, J9 Conn_02x10_Odd_Even, Q1 AO3401A, Q2 AO3401A, SW1 SW_Push, SW2 SW_Push, SW3 SW_Push, U1 AMS1117-3.3, U10 ATF22V10C-10PU, U11 SN74HC273DWR, U12 CD74HC4050M96, U13 SN74HCT574DWR, U14 FT230XS-U, U15 FE1.1S-BSOP28BCN, U16 MAX3421EETJ_T, U17 CD74HC4050M96, U18 SN76489AN, U19 SN76489AN, U2 LTC2954CTS8-2_TRMPBF, U20 LM386MX-1/NOPB, U21 SN74HCT574DWR, U22 TMS9928A, U23 THS7314DR, U24 AS7C256A-10TCN, U25 SN74LVC1G19DCKR, U26 SN74HC273DWR, U27 SN74HCT574DWR, U28 CD74HC139M96, U29 SN74HCT04DR, U3 ATmega1284-P, U30 SN74HC244DWR, U31 MAX202IDR, U4 SN74HC00ANSR, U5 SN74HC4040DR, U6 AS7C4096A-12TCN, U7 ATF22V10C-10PU, U8 Z084000xP, U9 SST39SF040-70-4C-PHE, Y1 ECS-2100AX-147.4, Y2 ABL-12.000MHZ-B2, Y3 ABL-12.000MHZ-B2, Y4 MP107-E

Commit message: Added pBITzBackplane and MezzanineConnector
Parts:
- removed the C2 at (1126.2, 54.6)
- added C2 (x2): 1000u, Capacitor_THT:CP_Radial_D10.0mm_P5.00mm, F.Cu at (58.1, 47.5)
- added C25: 100n, Capacitor_SMD:C_0603_1608Metric, F.Cu at (1126.5, 139.5)
- C1: value 10n -> 10u; footprint Capacitor_SMD:C_0805_2012Metric -> Capacitor_THT:CP_Radial_D5.0mm_P2.50mm
- C3: value 10u -> 100n; footprint Capacitor_SMD:C_0805_2012Metric -> Capacitor_SMD:C_0603_1608Metric
- C32, C38: footprint Capacitor_SMD:C_0603_1608Metric -> Capacitor_THT:CP_Radial_D5.0mm_P2.50mm
- C39, C40, C42, C51, C52, C53: footprint Capacitor_SMD:C_1206_3216Metric -> Capacitor_SMD:C_0603_1608Metric
- C41, C43, C46, C50: footprint Capacitor_Tantalum_SMD:CP_EIA-3528-21_Kemet-B -> Capacitor_THT:CP_Radial_D6.3mm_P2.50mm
- C6, C7: footprint Capacitor_SMD:C_0805_2012Metric -> Capacitor_SMD:C_0603_1608Metric
- D5, D6: value BAT54J -> BAT54JW-7-F
- J7: value Z80HomeBrewUser -> 1775862-2
- R15: value R -> 4k7
- R16: value R -> 10k
- RN1: value 4610X-101-103LF -> 4610X-101-472LF
- U3: value ATmega1284-P -> ATmega1284-PU
- moved J9 1100.5 mm to (1339.2, 16.4)
- moved Q2 1082.3 mm to (62.1, 37.0), turned to -90 degrees
- moved Q1 1082.3 mm to (62.1, 33.1), turned to 90 degrees
- moved F1 1079.0 mm to (60.6, 28.8)
- moved D2 1078.9 mm to (66.3, 28.0)
- moved D3 1078.4 mm to (66.3, 31.5), turned to -90 degrees
- moved R3 1075.9 mm to (59.7, 33.5), turned to -90 degrees
- moved R1 1075.9 mm to (59.6, 37.2), turned to 90 degrees
- moved C1 1073.0 mm to (66.6, 45.7), turned to 90 degrees
- moved R2 1070.8 mm to (64.7, 36.5), turned to 90 degrees
- moved D1 1070.7 mm to (74.2, 42.0)
- moved J1 1070.3 mm to (51.2, 38.4), turned to 90 degrees
- moved U2 1068.3 mm to (76.3, 35.7)
- moved C6 1066.3 mm to (73.5, 37.2), turned to -90 degrees
- moved R7 1066.1 mm to (69.9, 28.3), turned to -90 degrees
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Connections:
- C1 pad 1: Net-(Q1-S) -> +5V
- J6 pad 1: (no net) -> Net-(J13-Pin_1)
- J6 pad 2: (no net) -> Net-(J13-Pin_1)
- J6 pad 5: (no net) -> GND
- R35 pad 2: /CPU_AddressDecoding/~{INT} -> /Video/~{INT_}
- U22 pad 16: /CPU_AddressDecoding/~{INT} -> /Video/~{INT_}
- U25 pad 3: /CPU_AddressDecoding/~{INT} -> /Video/~{INT_}
Routing:
- net /CPU_AddressDecoding/D2: track 296.7 -> 381.0 mm, vias 8 -> 11
- net /CPU_AddressDecoding/D1: track 339.4 -> 423.6 mm, vias 10 -> 13
- net /CPU_AddressDecoding/D0: track 350.2 -> 433.5 mm, vias 11 -> 14
- net /CPU_AddressDecoding/D5: track 263.9 -> 338.0 mm, vias 10 -> 13
- net /CPU_AddressDecoding/A0: track 281.0 -> 348.3 mm, vias 5 -> 8
- net /CPU_AddressDecoding/D7: track 258.5 -> 325.2 mm, vias 8 -> 11
- net /CPU_AddressDecoding/A1: track 281.4 -> 344.8 mm, vias 5 -> 8
- net GND: track 95.1 -> 157.0 mm, vias 52 -> 92
- net /Video/AD7: track 0.00 -> 60.4 mm, vias 0 -> 3
- net /Video/AD6: track 0.00 -> 58.5 mm, vias 0 -> 3
- net /Video/AD5: track 0.00 -> 56.4 mm, vias 0 -> 3
- net Net-(U21-Q1): track 0.00 -> 56.4 mm, vias 0 -> 2
- net /Video/AD4: track 0.00 -> 54.7 mm, vias 0 -> 3
- net /Video/AD3: track 0.00 -> 52.4 mm, vias 0 -> 3
- net +5V: track 53.9 -> 105.5 mm, vias 21 -> 36
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- added copper zone on In2.Cu, net +3.3V
