File: Schem/Zephyr-80-CPU/IO Controller.kicad_sch (KiCad schematic)
At the start: 31 parts, among them IC1 Z80CTC, IC2 Z80SIO, IC3 Z80SIO, J5 Conn_01x08_Pin, SW1 SW_Push, SW2 SW_Push, U15 PIC18F57Q84-I/PT, U2 74AHC1G125, U3 74AHC1G125, U4 74AHC595, U5 74AHC595, U6 74HC138

Commit message: synching
Parts:
- removed J5: Conn_01x08_Pin, Connector_PinHeader_1.27mm:PinHeader_1x08_P1.27mm_Vertical, symbol Connector:Conn_01x08_Pin
- removed U15: PIC18F57Q84-I/PT, Footprints:TQFP48_PT_MCH, symbol 2026-02-07_23-07-57:PIC18F57Q84-I_PT
- added C1: 100n, Capacitor_SMD:C_0603_1608Metric, symbol Device:C
- added U1: ATmega1284-PU, Package_DIP:DIP-40_W15.24mm_Socket, symbol MCU_Microchip_ATmega:ATmega1284-P
Connections:
- net +5V: now also U1.10 (VCC), U1.30 (AVCC)
- net CTRL_LAT: now also U1.38 (PA2)
- net GND: now also C1.2, U1.11 (GND), U1.31 (GND)
- net GPIO0: now also U1.8 (PB7)
- net GPIO1: now also U1.7 (PB6)
- net GPIO2: now also U1.6 (PB5)
- net GPIO3: now also U1.5 (PB4)
- net GPIO4: now also U1.4 (PB3)
- net GPIO5: now also U1.3 (PB2)
- net GPIO6: now also U1.2 (PB1)
- net GPIO7: now also U1.1 (PB0)
- net RESET_HIGH: now also U1.21 (PD7)
- net SD_BUSY: now also U1.20 (PD6)
- net SD_PRESENT: now also U1.19 (PD5)
- net SPI_CLK: now also U1.29 (PC7)
- net SPI_MISO: now also U1.28 (PC6)
- net SPI_MOSI: now also U1.27 (PC5)
- net ~{CS_SIO_SD}: now also U1.22 (PC0)
- net ~{CS_SIO_USB}: now also U1.23 (PC1)
- net ~{NMI_RQ}: now also U1.17 (PD3)
- net ~{NMI}: now also U1.18 (PD4)
- net ~{POWER_OFF_RQ}: now also U1.14 (PD0)
- net ~{POWER_OFF}: now also U1.15 (PD1)
- net ~{RESET}: now also U1.16 (PD2)
- net ~{SD_CS}: now also U1.26 (PC4)
- net ~{SIO1A_INT}: now also U1.40 (PA0)
- net ~{SIO1B_INT}: now also U1.39 (PA1)
- net ~{USB_CS}: now also U1.25 (PC3)
- net ~{USB_INT}: now also U1.24 (PC2)
- net ~{MCLR}: no longer names the net of R1.2, SW1.2
- net ~{MCLR}: now also U1.9 (~{RESET})
- new net: C1.1, U1.32 (AREF)
- new net CLK_20M: U1.13 (XTAL1)
- no-connect marks 35 -> 24
Other:
- moved on the sheet: D1, IC1, IC2, IC3, R1, R2, SW1, SW2, U2, U3
