File: Schem/Zephyr-80-CPU/Zephyr-80-IO.kicad_sch (KiCad schematic)
At the start: 0 parts

Commit message: synching
Other:
- sheet IO Controller Card ports: added CLK_20M; removed none
- sheet pBITz Bus Interface ports: added CLK_20M; removed none
Changed lines of the file:
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@@
+	(wire
+		(pts
+			(xy 297.18 196.85) (xy 297.18 224.79)
+		)
+		(stroke
+			(width 0)
+			(type default)
+		)
+	)
 	(wire
 		(pts
@@
 			)
 		)
+		(pin "CLK_20M" input
+			(at 297.18 196.85 270)
+			(effects
+				(font
+					(size 1.27 1.27)
+				)
+				(justify left)
+			)
+		)
 		(pin "CLK_10M" input
 			(at 299.72 196.85 270)
@@
 			(effects
 				(font
+					(size 1.27 1.27)
+				)
+				(justify right)
+			)
+		)
+		(pin "CLK_20M" output
+			(at 297.18 224.79 90)
+			(effects
+				(font
