File: Schem/Zephyr-80-CPU/CPU_AddressDecoding.kicad_sch (KiCad schematic)
At the start: 17 parts, among them U1 AS7C4096A-12TCN, U2 ATF22V10C-10PU, U3 Z084000xP, U4 SST39SF040-70-4C-PHE, U5 ATF22V10C-10PU, U6 SN74HC273DWR, U7 SN74HC244DWR, Y1 ECS-2100AX-100

Commit message: Moved to the DIN Connector
Connections:
- net D0: now also U4.13 (DQ0); no longer U4.15 (DQ2)
- net D2: now also U4.15 (DQ2); no longer U4.13 (DQ0)
- net CS_SEL3: now reaches U2.20 (IO20)
- no-connect marks 12 -> 11
Changed lines of the file:
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@@
 	)
 	(no_connect
-		(at 229.87 63.5)
-	)
-	(no_connect
 		(at 199.39 78.74)
 	)
@@
 	(wire
 		(pts
+			(xy 229.87 63.5) (xy 240.03 63.5)
+		)
+		(stroke
+			(width 0)
+			(type default)
+		)
+	)
+	(wire
+		(pts
 			(xy 69.85 57.15) (xy 83.82 57.15)
 		)
@@
 		)
 	)
-	(label "D2"
+	(label "D0"
 		(at 295.91 184.15 0)
 		(effects
@@
 		)
 	)
-	(label "D0"
+	(label "D2"
 		(at 295.91 189.23 0)
 		(effects
@@
 		(effects
 			(font
+				(size 1.27 1.27)
+			)
+			(justify left)
+		)
+	)
+	(hierarchical_label "CS_SEL3"
+		(shape output)
+		(at 240.03 63.5 0)
+		(effects
+			(font

Commit message: Map ROM bits D5-D7 to the PLD to qualify RAM addresses
Connections:
- net ROM_A16: now also U5.18 (IO18)
- net ROM_A17: now also U5.19 (IO19)
- net ROM_A18: now also U5.20 (IO20)
- no-connect marks 11 -> 8
Changed lines of the file:
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@@
 	)
 	(no_connect
-		(at 231.14 162.56)
-	)
-	(no_connect
-		(at 231.14 165.1)
-	)
-	(no_connect
 		(at 199.39 81.28)
 	)
@@
 	)
 	(no_connect
-		(at 231.14 160.02)
-	)
-	(no_connect
 		(at 229.87 76.2)
 	)
@@
 	(wire
 		(pts
+			(xy 231.14 165.1) (xy 241.3 165.1)
+		)
+		(stroke
+			(width 0)
+			(type default)
+		)
+	)
+	(wire
+		(pts
 			(xy 295.91 186.69) (xy 313.69 186.69)
 		)
@@
 	(wire
 		(pts
+			(xy 231.14 162.56) (xy 241.3 162.56)
+		)
+		(stroke
+			(width 0)
+			(type default)
+		)
+	)
+	(wire
+		(pts
 			(xy 69.85 102.87) (xy 83.82 102.87)
 		)
@@
 	(wire
 		(pts
+			(xy 231.14 160.02) (xy 241.3 160.02)
+		)
+		(stroke
+			(width 0)
+			(type default)
+		)
+	)
+	(wire
+		(pts
 			(xy 190.5 157.48) (xy 200.66 157.48)
 		)
@@
 		)
 	)
+	(label "ROM_A16"
+		(at 241.3 165.1 180)
+		(effects
+			(font
+				(size 1.27 1.27)
+			)
+			(justify right bottom)
+		)
+	)
 	(label "D2"
 		(at 31.75 168.91 0)
@@
 	)
 	(label "ROM_A18"
+		(at 241.3 160.02 180)
+		(effects
+			(font
+				(size 1.27 1.27)
+			)
+			(justify right bottom)
+		)
+	)
+	(label "ROM_A18"
 		(at 295.91 153.67 0)
 		(effects
@@
 		)
 	)
+	(label "ROM_A17"
+		(at 241.3 162.56 180)
+		(effects
+			(font
+				(size 1.27 1.27)
+			)
+			(justify right bottom)
+		)
+	)
