File: Schem/pBITzBackplane/pBITzBackplane.kicad_pcb (KiCad board)
At the start: 4 copper layers, 243.8 x 243.8 mm, 71 parts, among them J1 ATX-24, J2 pBITzBus, J3 pBITzBus, J4 pBITzBus, J5 pBITzBus, J6 FH69-60S-0.5SH, J7 FH69-60S-0.5SH, Q1 BSS138, SW1 SW_Push, U1 ATtiny85-20P

Commit message: Major rework:
- Updated the Mezzanine to remove the slot connector and move it to the main board (facing the back)
-    The removal of the slot allowed for the removal of the FPC connector, which was a
     major source of complexity. The mezzanine now only has the SD card and USB connectors,
     which are much cheaper and easier to work with.
- The mezzanine is now more compact and cheaper to souirce

- The main board sees the addition of the external slot connector (coming from the mezzanine)
- Added power led on the mother board for easier debugging and testing
- Removed the free floating resistors to replace them with resistor packs
Parts:
- removed ?: OSHW-Logo2_7.3x6mm_SilkScreen, Symbol:OSHW-Logo2_7.3x6mm_SilkScreen
- removed R10, R11, R12, R13, R14, R15, R16, R17, R6, R7, R9: 4k7, Resistor_SMD:R_0603_1608Metric
- removed RN10, RN11, RN12, RN13, RN14, RN15, RN5, RN6, RN7, RN8, RN9: EXB-2HV330JV, Footprints:RESCAXE50P380X160X55-16N
- added C16: 100n, Capacitor_SMD:C_0603_1608Metric, F.Cu at (278.5, 223.6)
- added C17: 100n, Capacitor_SMD:C_0603_1608Metric, F.Cu at (278.5, 226.1)
- added D1: LED, LED_THT:LED_D5.0mm, F.Cu at (330.6, 383.6)
- added D2: LED, Connector_PinHeader_2.54mm:PinHeader_2x01_P2.54mm_Vertical, F.Cu at (324.6, 383.5)
- added R19: 4k7, Resistor_SMD:R_0603_1608Metric, F.Cu at (324.6, 386.3)
- added R20: 4k7, Resistor_SMD:R_0603_1608Metric, F.Cu at (330.5, 386.3)
- J6: value FH69-60S-0.5SH -> pBITzBus; footprint Footprints:CONN60_FH69-60S_HIR -> Footprints:SAMTEC_PCIE-098-02-X-D-RA
- J7: value FH69-60S-0.5SH -> Conn_02x10_Odd_Even; footprint Footprints:CONN60_FH69-60S_HIR -> Connector_IDC:IDC-Header_2x10_P2.54mm_Vertical
- RN4: value EXB-2HV330JV -> 4816P-T02-472LF; footprint Footprints:RESCAXE50P380X160X55-16N -> Footprints:4816PT02472LF
- moved J6 78.4 mm to (308.5, 216.9), turned to 180 degrees
- moved RN4 65.8 mm to (310.0, 292.1)
- moved RN1 56.3 mm to (295.8, 292.1), turned to 90 degrees
- moved H10 51.1 mm to (293.1, 352.7)
- moved H11 50.4 mm to (202.2, 352.7)
- moved J7 33.4 mm to (251.8, 327.9), turned to 90 degrees
- moved RN3 30.9 mm to (323.3, 292.0), turned to 90 degrees
- moved H12 20.7 mm to (293.1, 424.1)
- moved G*** 20.1 mm to (235.9, 387.9)
- moved H13 18.8 mm to (202.2, 424.1)
- moved RN2 16.8 mm to (337.3, 292.0), turned to 90 degrees
Connections:
- J7 pad 1: GND -> +5V
- J7 pad 10: /Backplane/CART_T -> GND
- J7 pad 11: +3V3 -> GND
- J7 pad 12: +3V3 -> unconnected-(J7-Pin_12-Pad12)
- J7 pad 13: /Backplane/~{RESET_T} -> /Backplane/~{SPI_INT}
- J7 pad 14: /Backplane/CTRL_1_T -> GND
- J7 pad 15: /Backplane/CTRL_2_T -> GND
- J7 pad 16: /Backplane/CTRL_3_T -> GND
- J7 pad 17: /Backplane/CTRL_4_T -> /Backplane/SPI_CD
- J7 pad 18: /Backplane/CTRL_5_T -> GND
- J7 pad 19: /Backplane/CTRL_6_T -> GND
- J7 pad 2: +5V -> +3V3
- J7 pad 20: /Backplane/CTRL_7_T -> GND
- J7 pad 3: +5V -> /Backplane/MOSI
- J7 pad 4: unconnected-(J7-Pad4) -> /Backplane/SPI_CS0
- J7 pad 5: GND -> /Backplane/MISO
- J7 pad 6: /Backplane/CLK0_T -> GND
- J7 pad 7: /Backplane/CLK1_T -> GND
- J7 pad 8: GND -> /Backplane/SPI_CS1
- J7 pad 9: /Backplane/SPI_CD_T -> /Backplane/SLK_CLK
- RN1 pad 1: /Backplane/CTRL_10 -> /Backplane/CART
- RN1 pad 10: /Backplane/CTRL_19 -> /Backplane/CTRL_8
- RN1 pad 11: /Backplane/CTRL_9 -> /Backplane/CTRL_17
- RN1 pad 12: /Backplane/CTRL_8 -> /Backplane/CTRL_16
- RN1 pad 13: /Backplane/CTRL_7 -> /Backplane/CTRL_15
- RN1 pad 14: /Backplane/CTRL_6 -> /Backplane/CTRL_14
- RN1 pad 15: /Backplane/CTRL_5 -> /Backplane/CTRL_13
- RN1 pad 16: /Backplane/CTRL_4 -> /Backplane/CTRL_12
- RN1 pad 17: /Backplane/CTRL_3 -> /Backplane/CTRL_11
- RN1 pad 18: /Backplane/CTRL_2 -> /Backplane/CTRL_10
- RN1 pad 19: /Backplane/CTRL_1 -> /Backplane/PROG
- RN1 pad 2: /Backplane/CTRL_11 -> /Backplane/~{RESET}
- RN1 pad 3: /Backplane/CTRL_12 -> /Backplane/CTRL_1
- RN1 pad 4: /Backplane/CTRL_13 -> /Backplane/CTRL_2
- RN1 pad 5: /Backplane/CTRL_14 -> /Backplane/CTRL_3
- RN1 pad 6: /Backplane/CTRL_15 -> /Backplane/CTRL_4
- RN1 pad 7: /Backplane/CTRL_16 -> /Backplane/CTRL_5
- RN1 pad 8: /Backplane/CTRL_17 -> /Backplane/CTRL_6
- RN1 pad 9: /Backplane/CTRL_18 -> /Backplane/CTRL_7
- RN2 pad 1: /Backplane/A12 -> /Backplane/A15
- RN2 pad 10: /Backplane/A21 -> unconnected-(RN2-Pad10)
- RN2 pad 11: /Backplane/A8 -> unconnected-(RN2-Pad11)
- RN2 pad 12: /Backplane/A7 -> /Backplane/A20
- RN2 pad 13: /Backplane/A6 -> /Backplane/A21
- RN2 pad 14: /Backplane/A5 -> /Backplane/A22
- RN2 pad 15: /Backplane/A4 -> /Backplane/A23
- RN2 pad 16: /Backplane/A3 -> /Backplane/A7
- RN2 pad 17: /Backplane/A2 -> /Backplane/A6
- RN2 pad 18: /Backplane/A1 -> /Backplane/A5
- RN2 pad 19: /Backplane/A0 -> /Backplane/A4
- RN2 pad 2: /Backplane/A13 -> /Backplane/A16
- RN2 pad 3: /Backplane/A14 -> /Backplane/A17
- RN2 pad 4: /Backplane/A15 -> /Backplane/A18
- RN2 pad 5: /Backplane/A16 -> /Backplane/A19
- RN2 pad 6: /Backplane/A17 -> /Backplane/A11
- RN2 pad 7: /Backplane/A18 -> /Backplane/A10
- RN2 pad 8: /Backplane/A19 -> /Backplane/A9
- RN2 pad 9: /Backplane/A20 -> /Backplane/A8
- RN3 pad 1: /Backplane/D8 -> /Backplane/D4
- RN3 pad 10: /Backplane/D5 -> /Backplane/A2
- RN3 pad 11: /Backplane/D4 -> /Backplane/A1
- RN3 pad 12: /Backplane/D3 -> /Backplane/A0
- RN3 pad 13: /Backplane/D2 -> /Backplane/D7
- RN3 pad 14: /Backplane/D1 -> /Backplane/D6
- RN3 pad 15: /Backplane/D0 -> /Backplane/D5
- RN3 pad 2: /Backplane/D9 -> /Backplane/D12
- RN3 pad 3: /Backplane/D10 -> /Backplane/D13
- RN3 pad 4: /Backplane/D11 -> /Backplane/D14
- RN3 pad 5: /Backplane/D12 -> /Backplane/D15
- RN3 pad 6: /Backplane/D13 -> /Backplane/A12
- RN3 pad 7: /Backplane/D14 -> /Backplane/A13
- RN3 pad 8: /Backplane/D15 -> /Backplane/A14
- RN3 pad 9: /Backplane/D6 -> /Backplane/A3
- RN4 pad 1: /Backplane/SPI_CS1_T -> /Backplane/CTRL_18
- RN4 pad 10: /Backplane/A10 -> /Backplane/D10
- RN4 pad 11: /Backplane/A11 -> /Backplane/D9
- RN4 pad 12: unconnected-(RN4-Pad12) -> /Backplane/D8
- RN4 pad 13: unconnected-(RN4-Pad13) -> /Backplane/CS3
- RN4 pad 14: /Backplane/MOSI -> /Backplane/CS2
- RN4 pad 15: unconnected-(RN4-Pad15) -> /Backplane/CS0
- RN4 pad 16: /Backplane/SPI_CS1 -> +5V
- RN4 pad 2: unconnected-(RN4-Pad2) -> /Backplane/CTRL_9
- RN4 pad 3: /Backplane/MOSI_T -> /Backplane/CTRL_19
- RN4 pad 4: unconnected-(RN4-Pad4) -> /Backplane/CS1
- RN4 pad 5: unconnected-(RN4-Pad5) -> /Backplane/D0
- RN4 pad 6: /Backplane/A11_T -> /Backplane/D1
- RN4 pad 7: /Backplane/A10_T -> /Backplane/D2
- RN4 pad 8: /Backplane/A9_T -> /Backplane/D3
- RN4 pad 9: /Backplane/A9 -> /Backplane/D11
Routing:
- net /Backplane/SPI_CS1: track 82.9 -> 282.5 mm
- net /Backplane/MOSI: track 85.2 -> 279.9 mm, vias 1 -> 3
- net /Backplane/SPI_CS0: track 120.3 -> 281.5 mm, vias 2 -> 1
- net /Backplane/MISO: track 120.2 -> 279.6 mm, vias 2 -> 3
- net /Backplane/~{SPI_INT}: track 124.3 -> 281.5 mm, vias 2 -> 3
- net /Backplane/SPI_CD: track 148.3 -> 241.1 mm, vias 1 -> 2
- net /Backplane/A23: track 165.3 -> 233.6 mm, vias 3 -> 2
- net /Backplane/A21: track 167.7 -> 235.3 mm, vias 3 -> 2
- net /Backplane/A22: track 167.9 -> 234.3 mm, vias 3 -> 2
- net /Backplane/A20: track 169.0 -> 234.9 mm, vias 3 -> 2
- net /Backplane/A19: track 171.9 -> 237.5 mm, vias 3 -> 2
- net /Backplane/A18: track 171.3 -> 236.7 mm, vias 3 -> 2
- net /Backplane/A17: track 172.9 -> 235.9 mm, vias 3 -> 2
- net /Backplane/SLK_CLK: track 188.0 -> 250.7 mm
- net /Backplane/A10: track 182.8 -> 245.3 mm
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Other:
- board text removed: "A0"
- board text removed: "A11"
- board text removed: "A8"
- board text removed: "CS0"
- board text removed: "D0"
- board text removed: "D7"
- board text removed: "Expansion Connector (A-Side)"
- board text removed: "Expansion Connector (B-Side)"
