File: Schem/pBITzBackplane/pBITzBackplane.kicad_sch (KiCad schematic)
At the start: 13 parts

Commit message: Fixed board
Parts:
- H1: value MountingHole (F) -> MountingHole; footprint MountingHole:MountingHole_3.2mm_M3_Pad_Via -> MountingHole:MountingHole_3.5mm_Pad_TopBottom
- H10, H11, H12, H13, H2, H3, H4, H5, H6, H7, H8, H9: footprint MountingHole:MountingHole_3.2mm_M3_Pad_Via -> MountingHole:MountingHole_3.5mm_Pad_TopBottom
Other:
- sheet Backplane ports: added ~{SHUTDOWN_RQ}; removed ~{PWR_OFF_RQ}
- sheet Power ports: added ~{PWR_OFF}, ~{SHUTDOWN_RQ}; removed PWR_OFF_RQ, PWR_STATE
- moved on the sheet: H11, H13, H2, H4, H6, H8
