File: Schem/pBITzBackplane/Backplane.kicad_sch (KiCad schematic)
At the start: 40 parts, among them J2 pBITzBus, J3 pBITzBus, J4 pBITzBus, J5 pBITzBus, J6 FH69-60S-0.5SH, J7 FH69-60S-0.5SH

Commit message: Major rework:
- Updated the Mezzanine to remove the slot connector and move it to the main board (facing the back)
-    The removal of the slot allowed for the removal of the FPC connector, which was a
     major source of complexity. The mezzanine now only has the SD card and USB connectors,
     which are much cheaper and easier to work with.
- The mezzanine is now more compact and cheaper to souirce

- The main board sees the addition of the external slot connector (coming from the mezzanine)
- Added power led on the mother board for easier debugging and testing
- Removed the free floating resistors to replace them with resistor packs
Parts:
- removed J6, J7: FH69-60S-0.5SH, Footprints:CONN60_FH69-60S_HIR, symbol 2026-01-31_22-05-17:FH69-60S-0.5SH
- removed R10, R11, R12, R13, R14, R15, R16, R17, R6, R7, R9: 4k7, Resistor_SMD:R_0603_1608Metric, symbol Device:R
- removed RN10, RN11, RN12, RN13, RN14, RN15, RN4, RN5, RN6, RN7, RN8, RN9: EXB-2HV330JV, Footprints:RESCAXE50P380X160X55-16N, symbol EXB-2HV330JV:EXB-2HV330JV
- added C16, C17: 100n, Capacitor_SMD:C_0603_1608Metric, symbol Device:C
- added J6: pBITzBus, Footprints:SAMTEC_PCIE-098-02-X-D-RA, symbol pBITz:pBITzBus
- added J7: Conn_02x10_Odd_Even, Connector_IDC:IDC-Header_2x10_P2.54mm_Vertical, symbol Connector_Generic:Conn_02x10_Odd_Even
- added RN4: 4816P-T02-472LF, Footprints:4816PT02472LF, symbol 4816P-T02-472LF:4816P-T02-472LF
- C10, C11, C12, C13, C14, C15, C8, C9: MANUFACTURER_PART_NUMBER (none) -> C0603C104K3RACTU
- J5: MANUFACTURER_PART_NUMBER PCIE-098-02-F-D-RA -> 10018783-10202TLF
- RN1, RN2: Manufacturer_Part_Number 4820P-2-472LF -> (none)
- RN3: Manufacturer_Part_Number 4816P-T02-472LF -> (none)
Connections:
- net +3V3: now also C16.1, J6.A10 (+3V3), J6.A9 (+3V3), J6.B10 (+3V3), J6.B9 (+3V3), J7.2 (Pin_2)
- net +5V: now also C17.1, J6.A1 (+5V), J6.A2 (+5V), J6.B1 (+5V), J6.B2 (+5V), J7.1 (Pin_1), RN4.16
- net A0: now also RN3.12, J6.B32 (A0); no longer RN2.19
- net A1: now also RN3.11, J6.B33 (A1); no longer RN2.18
- net A10: now also RN2.7, J6.B45 (A10)
- net A11: now also RN2.6, J6.B46 (A11)
- net A12: now also RN3.6, J6.A32 (A12); no longer RN2.1
- net A13: now also RN3.7, J6.A33 (A13); no longer RN2.2
- net A14: now also RN3.8, J6.A34 (A14); no longer RN2.3
- net A15: now also RN2.1, J6.A36 (A15); no longer RN2.4
- net A16: now also RN2.2, J6.A37 (A16); no longer RN2.5
- net A17: now also RN2.3, J6.A38 (A17); no longer RN2.6
- net A18: now also RN2.4, J6.A40 (A18); no longer RN2.7
- net A19: now also RN2.5, J6.A41 (A19); no longer RN2.8
- net A2: now also RN3.10, J6.B34 (A2); no longer RN2.17
- net A20: now also RN2.12, J6.A42 (A20); no longer RN2.9
- net A21: now also RN2.13, J6.A44 (A21); no longer RN2.10
- net A22: now also RN2.14, J6.A45 (A22)
- net A23: now also RN2.15, J6.A46 (A23)
- net A3: now also RN3.9, J6.B36 (A3); no longer RN2.16
- net A4: now also RN2.19, J6.B37 (A4); no longer RN2.15
- net A5: now also RN2.18, J6.B38 (A5); no longer RN2.14
- net A6: now also RN2.17, J6.B40 (A6); no longer RN2.13
- net A7: now also RN2.16, J6.B41 (A7); no longer RN2.12
- net A8: now also RN2.9, J6.B42 (A8); no longer RN2.11
- net A9: now also RN2.8, J6.B44 (A9)
- net CART: now also RN1.1, J6.B8 (CART)
- net CLK0: now also J6.B5 (CLK0)
- net CLK1: now also J6.B6 (CLK1)
- net CLK2: now also J6.A5 (CLK2)
- net CLK3: now also J6.A6 (CLK3)
- net CS0: now also J6.B21 (CS0), RN4.15
- net CS1: now also J6.B22 (CS1), RN4.4
- net CS2: now also J6.A21 (CS2), RN4.14
- net CS3: now also J6.A22 (CS3), RN4.13
- net CTRL_1: now also RN1.3, J6.B12 (CTRL_1); no longer RN1.19
- net CTRL_10: now also RN1.18, J6.A11 (CTRL_10); no longer RN1.1
- net CTRL_11: now also RN1.17, J6.A12 (CTRL_11); no longer RN1.2
- net CTRL_12: now also RN1.16, J6.A13 (CTRL_12); no longer RN1.3
- net CTRL_13: now also RN1.15, J6.A14 (CTRL_13); no longer RN1.4
- net CTRL_14: now also RN1.14, J6.A15 (CTRL_14); no longer RN1.5
- net CTRL_15: now also RN1.13, J6.A16 (CTRL_15); no longer RN1.6
- net CTRL_16: now also RN1.12, J6.A17 (CTRL_16); no longer RN1.7
- net CTRL_17: now also RN1.11, J6.A18 (CTRL_17); no longer RN1.8
- net CTRL_18: now also J6.A19 (CTRL_18), RN4.1; no longer RN1.9
- net CTRL_19: now also J6.A20 (CTRL_19), RN4.3; no longer RN1.10
- net CTRL_2: now also RN1.4, J6.B13 (CTRL_2); no longer RN1.18
- net CTRL_3: now also RN1.5, J6.B14 (CTRL_3); no longer RN1.17
- net CTRL_4: now also RN1.6, J6.B15 (CTRL_4); no longer RN1.16
- net CTRL_5: now also RN1.7, J6.B16 (CTRL_5); no longer RN1.15
- net CTRL_6: now also RN1.8, J6.B17 (CTRL_6); no longer RN1.14
- net CTRL_7: now also RN1.9, J6.B18 (CTRL_7); no longer RN1.13
- net CTRL_8: now also RN1.10, J6.B19 (CTRL_8); no longer RN1.12
- net CTRL_9: now also J6.B20 (CTRL_9), RN4.2; no longer RN1.11
- net D0: now also J6.B23 (D0), RN4.5; no longer RN3.15
- net D1: now also J6.B24 (D1), RN4.6; no longer RN3.14
- net D10: now also J6.A25 (D10), RN4.10; no longer RN3.3
- net D11: now also J6.A26 (D11), RN4.9; no longer RN3.4
- net D12: now also RN3.2, J6.A27 (D12); no longer RN3.5
- net D13: now also RN3.3, J6.A28 (D13); no longer RN3.6
- net D14: now also RN3.4, J6.A29 (D14); no longer RN3.7
- net D15: now also RN3.5, J6.A30 (D15); no longer RN3.8
- net D2: now also J6.B25 (D2), RN4.7; no longer RN3.13
- net D3: now also J6.B26 (D3), RN4.8; no longer RN3.12
- net D4: now also RN3.1, J6.B27 (D4); no longer RN3.11
- net D5: now also RN3.15, J6.B28 (D5); no longer RN3.10
- net D6: now also RN3.14, J6.B29 (D6); no longer RN3.9
- net D7: now also RN3.13, J6.B30 (D7)
- net D8: now also J6.A23 (D8), RN4.12; no longer RN3.1
- net D9: now also J6.A24 (D9), RN4.11; no longer RN3.2
- net GND: now also C16.2, C17.2, J6.A31 (GND), J6.A35 (GND), J6.A39 (GND), J6.A4 (GND), J6.A43 (GND), J6.B31 (GND), J6.B35 (GND), J6.B39 (GND), J6.B4 (GND), J6.B43 (GND), J6.B47 (GND), J7.10 (Pin_10), J7.11 (Pin_11), J7.14 (Pin_14), J7.15 (Pin_15), J7.16 (Pin_16), J7.18 (Pin_18), J7.19 (Pin_19), J7.20 (Pin_20), J7.6 (Pin_6), J7.7 (Pin_7)
- net MISO: now also J6.A48 (MISO), J7.5 (Pin_5)
- net MOSI: now also J6.B48 (MOSI), J7.3 (Pin_3)
- net PROG: now also RN1.19, J6.A8 (PROG)
- net SLK_CLK: now also J6.A7 (SPI_CLK), J7.9 (Pin_9)
- net SPI_CD: now also J6.B7 (SPI_CD), J7.17 (Pin_17)
- net SPI_CS0: now also J6.A49 (SPI_CS0), J7.4 (Pin_4)
- net SPI_CS1: now also J6.B49 (SPI_CS1), J7.8 (Pin_8)
- net ~{PWR_OFF_RQ}: now also J6.A3 (~{PWR_OFF_RQ})
- net ~{PWR_OFF}: now also J6.B3 (~{PWR_OFF})
- net ~{RESET}: now also RN1.2, J6.B11 (CTRL_0)
- net ~{SPI_INT}: now also J6.A47 (~{SPI_INT}), J7.13 (Pin_13)
- no-connect marks 40 -> 3

Commit message: Fixed board
Parts:
- C10, C11, C12, C13, C14, C15, C16, C17, C8, C9: footprint Capacitor_SMD:C_0603_1608Metric -> Capacitor_SMD:C_1206_3216Metric
Connections:
- net ~{PWR_OFF_RQ} renamed ~{SHUTDOWN_RQ}
Changed lines of the file:
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@@
 		)
 	)
-	(hierarchical_label "~{PWR_OFF_RQ}"
-		(shape input)
-		(at 107.95 351.79 180)
+	(hierarchical_label "~{PWR_OFF}"
+		(shape output)
+		(at 81.28 351.79 0)
 		(effects
 			(font
 				(size 1.27 1.27)
 			)
-			(justify right)
+			(justify left)
 		)
 	)
-	(hierarchical_label "~{PWR_OFF_RQ}"
+	(hierarchical_label "~{SHUTDOWN_RQ}"
 		(shape input)
-		(at 334.01 351.79 180)
+		(at 256.54 351.79 180)
 		(effects
 			(font
@@
 		)
 	)
-	(hierarchical_label "~{PWR_OFF}"
-		(shape output)
-		(at 81.28 351.79 0)
-		(effects
-			(font
-				(size 1.27 1.27)
-			)
-			(justify left)
-		)
-	)
-	(hierarchical_label "~{PWR_OFF_RQ}"
+	(hierarchical_label "~{SHUTDOWN_RQ}"
 		(shape input)
-		(at 182.88 351.79 180)
+		(at 33.02 351.79 180)
 		(effects
 			(font
@@
 		)
 	)
-	(hierarchical_label "~{PWR_OFF_RQ}"
+	(hierarchical_label "~{SHUTDOWN_RQ}"
 		(shape input)
-		(at 33.02 351.79 180)
+		(at 107.95 351.79 180)
 		(effects
 			(font
@@
 		)
 	)
-	(hierarchical_label "~{PWR_OFF}"
-		(shape output)
-		(at 304.8 351.79 0)
+	(hierarchical_label "~{SHUTDOWN_RQ}"
+		(shape input)
+		(at 334.01 351.79 180)
 		(effects
 			(font
 				(size 1.27 1.27)
 			)
-			(justify left)
+			(justify right)
 		)
 	)
-	(hierarchical_label "~{PWR_OFF_RQ}"
-		(shape input)
-		(at 256.54 351.79 180)
+	(hierarchical_label "~{PWR_OFF}"
+		(shape output)
+		(at 304.8 351.79 0)
 		(effects
 			(font
 				(size 1.27 1.27)
 			)
-			(justify right)
+			(justify left)
 		)
 	)
@@
 		)
 	)
+	(hierarchical_label "~{SHUTDOWN_RQ}"
+		(shape input)
+		(at 182.88 351.79 180)
+		(effects
+			(font
+				(size 1.27 1.27)
+			)
+			(justify right)
+		)
+	)
 	(hierarchical_label "~{PWR_OFF}"
 		(shape output)
@@
 			)
 		)
-		(property "Footprint" "Capacitor_SMD:C_0603_1608Metric"
+		(property "Footprint" "Capacitor_SMD:C_1206_3216Metric"
 			(at 55.5752 393.7 0)
 			(hide yes)
@@
 			)
 		)
-		(property "Footprint" "Capacitor_SMD:C_0603_1608Metric"
+		(property "Footprint" "Capacitor_SMD:C_1206_3216Metric"
 			(at 44.1452 393.7 0)
 			(hide yes)
@@
 	)
 	(symbol
+		(lib_name "pBITzBus_11")
 		(lib_id "pBITz:pBITzBus")
 		(at 207.01 384.81 0)
@@
 			)
 		)
-		(property "Footprint" "Capacitor_SMD:C_0603_1608Metric"
+		(property "Footprint" "Capacitor_SMD:C_1206_3216Metric"
 			(at 101.2952 393.7 0)
 			(hide yes)
@@
 			)
 		)
-		(property "Footprint" "Capacitor_SMD:C_0603_1608Metric"
+		(property "Footprint" "Capacitor_SMD:C_1206_3216Metric"
 			(at 133.0452 393.7 0)
 			(hide yes)
@@
 			)
 		)
-		(property "Footprint" "Capacitor_SMD:C_0603_1608Metric"
+		(property "Footprint" "Capacitor_SMD:C_1206_3216Metric"
 			(at 147.0152 393.7 0)
 			(hide yes)
@@
 			)
 		)
-		(property "Footprint" "Capacitor_SMD:C_0603_1608Metric"
+		(property "Footprint" "Capacitor_SMD:C_1206_3216Metric"
 			(at 116.5352 393.7 0)
 			(hide yes)
@@
 	)
 	(symbol
+		(lib_name "pBITzBus_9")
 		(lib_id "pBITz:pBITzBus")
 		(at 57.15 384.81 0)
@@
 	)
 	(symbol
+		(lib_name "pBITzBus_10")
 		(lib_id "pBITz:pBITzBus")
 		(at 132.08 384.81 0)
@@
 			)
 		)
-		(property "Footprint" "Capacitor_SMD:C_0603_1608Metric"
+		(property "Footprint" "Capacitor_SMD:C_1206_3216Metric"
 			(at 86.0552 393.7 0)
 			(hide yes)
@@
 			)
 		)
-		(property "Footprint" "Capacitor_SMD:C_0603_1608Metric"
+		(property "Footprint" "Capacitor_SMD:C_1206_3216Metric"
 			(at 160.9852 393.7 0)
 			(hide yes)
@@
 			)
 		)
-		(property "Footprint" "Capacitor_SMD:C_0603_1608Metric"
+		(property "Footprint" "Capacitor_SMD:C_1206_3216Metric"
 			(at 173.6852 393.7 0)
 			(hide yes)
@@
 	)
 	(symbol
+		(lib_name "pBITzBus_12")
 		(lib_id "pBITz:pBITzBus")
 		(at 280.67 384.81 0)
@@
 			)
 		)
-		(property "Footprint" "Capacitor_SMD:C_0603_1608Metric"
+		(property "Footprint" "Capacitor_SMD:C_1206_3216Metric"
 			(at 69.5452 393.7 0)
 			(hide yes)

Commit message: Made the footprint bigger to facilitate soldering.
Parts:
- C10, C11, C12, C13, C14, C15, C16, C17, C8, C9: footprint Capacitor_SMD:C_1206_3216Metric -> Capacitor_SMD:C_1206_3216Metric_Pad1.33x1.80mm_HandSolder
Changed lines of the file:
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@@
 			)
 		)
-		(property "Footprint" "Capacitor_SMD:C_1206_3216Metric"
+		(property "Footprint" "Capacitor_SMD:C_1206_3216Metric_Pad1.33x1.80mm_HandSolder"
 			(at 55.5752 393.7 0)
 			(hide yes)
@@
 			)
 		)
-		(property "Footprint" "Capacitor_SMD:C_1206_3216Metric"
+		(property "Footprint" "Capacitor_SMD:C_1206_3216Metric_Pad1.33x1.80mm_HandSolder"
 			(at 44.1452 393.7 0)
 			(hide yes)
@@
 			)
 		)
-		(property "Footprint" "Capacitor_SMD:C_1206_3216Metric"
+		(property "Footprint" "Capacitor_SMD:C_1206_3216Metric_Pad1.33x1.80mm_HandSolder"
 			(at 101.2952 393.7 0)
 			(hide yes)
@@
 			)
 		)
-		(property "Footprint" "Capacitor_SMD:C_1206_3216Metric"
+		(property "Footprint" "Capacitor_SMD:C_1206_3216Metric_Pad1.33x1.80mm_HandSolder"
 			(at 133.0452 393.7 0)
 			(hide yes)
@@
 			)
 		)
-		(property "Footprint" "Capacitor_SMD:C_1206_3216Metric"
+		(property "Footprint" "Capacitor_SMD:C_1206_3216Metric_Pad1.33x1.80mm_HandSolder"
 			(at 147.0152 393.7 0)
 			(hide yes)
@@
 			)
 		)
-		(property "Footprint" "Capacitor_SMD:C_1206_3216Metric"
+		(property "Footprint" "Capacitor_SMD:C_1206_3216Metric_Pad1.33x1.80mm_HandSolder"
 			(at 116.5352 393.7 0)
 			(hide yes)
@@
 			)
 		)
-		(property "Footprint" "Capacitor_SMD:C_1206_3216Metric"
+		(property "Footprint" "Capacitor_SMD:C_1206_3216Metric_Pad1.33x1.80mm_HandSolder"
 			(at 86.0552 393.7 0)
 			(hide yes)
@@
 			)
 		)
-		(property "Footprint" "Capacitor_SMD:C_1206_3216Metric"
+		(property "Footprint" "Capacitor_SMD:C_1206_3216Metric_Pad1.33x1.80mm_HandSolder"
 			(at 160.9852 393.7 0)
 			(hide yes)
@@
 			)
 		)
-		(property "Footprint" "Capacitor_SMD:C_1206_3216Metric"
+		(property "Footprint" "Capacitor_SMD:C_1206_3216Metric_Pad1.33x1.80mm_HandSolder"
 			(at 173.6852 393.7 0)
 			(hide yes)
@@
 			)
 		)
-		(property "Footprint" "Capacitor_SMD:C_1206_3216Metric"
+		(property "Footprint" "Capacitor_SMD:C_1206_3216Metric_Pad1.33x1.80mm_HandSolder"
 			(at 69.5452 393.7 0)
 			(hide yes)

Commit message: Fixed part #s
Parts:
- J2, J3, J4: MANUFACTURER_PART_NUMBER PCIE-098-02-F-D-RA -> 10018783-10202TLF
Changed lines of the file:
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@@
 			)
 		)
-		(property "MANUFACTURER_PART_NUMBER" "PCIE-098-02-F-D-RA"
+		(property "MANUFACTURER_PART_NUMBER" "10018783-10202TLF"
 			(at 57.15 308.61 0)
 			(hide yes)
@@
 			)
 		)
-		(property "MANUFACTURER_PART_NUMBER" "PCIE-098-02-F-D-RA"
+		(property "MANUFACTURER_PART_NUMBER" "10018783-10202TLF"
 			(at 57.15 384.81 0)
 			(hide yes)
@@
 			)
 		)
-		(property "MANUFACTURER_PART_NUMBER" "PCIE-098-02-F-D-RA"
+		(property "MANUFACTURER_PART_NUMBER" "10018783-10202TLF"
 			(at 132.08 384.81 0)
 			(hide yes)
@@
 			)
 		)
-		(property "MANUFACTURER_PART_NUMBER" "PCIE-098-02-F-D-RA"
+		(property "MANUFACTURER_PART_NUMBER" "10018783-10202TLF"
 			(at 293.37 92.71 0)
 			(hide yes)
@@
 			)
 		)
-		(property "MANUFACTURER_PART_NUMBER" "PCIE-098-02-F-D-RA"
+		(property "MANUFACTURER_PART_NUMBER" "10018783-10202TLF"
 			(at 144.78 308.61 0)
 			(hide yes)
@@
 			)
 		)
-		(property "MANUFACTURER_PART_NUMBER" "PCIE-098-02-F-D-RA"
+		(property "MANUFACTURER_PART_NUMBER" "10018783-10202TLF"
 			(at 100.33 308.61 0)
 			(hide yes)
@@
 			)
 		)
-		(property "MANUFACTURER_PART_NUMBER" "PCIE-098-02-F-D-RA"
+		(property "MANUFACTURER_PART_NUMBER" "10018783-10202TLF"
 			(at 199.39 92.71 0)
 			(hide yes)
@@
 			)
 		)
-		(property "MANUFACTURER_PART_NUMBER" "PCIE-098-02-F-D-RA"
+		(property "MANUFACTURER_PART_NUMBER" "10018783-10202TLF"
 			(at 280.67 384.81 0)
 			(hide yes)
@@
 			)
 		)
-		(property "MANUFACTURER_PART_NUMBER" "PCIE-098-02-F-D-RA"
+		(property "MANUFACTURER_PART_NUMBER" "10018783-10202TLF"
 			(at 96.52 93.98 0)
 			(hide yes)
