File: Schem/Zephyr-80-IO/BaudClock.kicad_sch (KiCad schematic)
At the start: 3 parts, among them U8 SN74HC4040DR, Y1 ECS-2100AX-147.4

Commit message: updated parts #s
Parts:
- U8: MANUFACTURER_PART_NUMBER MC74HC4040ADTR2G -> SN74HC4040PWR
Changed lines of the file:
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@@
 			)
 		)
-		(property "MANUFACTURER_PART_NUMBER" "MC74HC4040ADTR2G"
+		(property "MANUFACTURER_PART_NUMBER" "SN74HC4040PWR"
 			(at 134.62 74.93 0)
 			(hide yes)
