File: Schem/Zephyr-80-IO/DeviceSelectDecode.kicad_sch (KiCad schematic)
At the start: 29 parts, among them SW3 SW_Coded_SH-7070, SW4 SW_Coded_SH-7070, SW5 SW_Coded_SH-7070, SW6 SW_Coded_SH-7070, U10 74HC688, U11 74HC688, U12 74HC688, U9 74HC688

Commit message: Moved to the DIN Connector
Connections:
- net GND: no longer U10.1 (G)
- new net ~{RD}: U10.1 (G)
Changed lines of the file:
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@@
-	)
-	(junction
-		(at 255.27 135.89)
-		(diameter 0)
-		(color 0 0 0 0)
 	)
 	(junction
@@
 	(wire
 		(pts
+			(xy 251.46 135.89) (xy 259.08 135.89)
+		)
+		(stroke
+			(width 0)
+			(type default)
+		)
+	)
+	(wire
+		(pts
 			(xy 508 106.68) (xy 511.81 106.68)
 		)
@@
 	(wire
 		(pts
-			(xy 255.27 135.89) (xy 259.08 135.89)
-		)
-		(stroke
-			(width 0)
-			(type default)
-		)
-	)
-	(wire
-		(pts
 			(xy 255.27 105.41) (xy 255.27 107.95)
 		)
@@
 	(wire
 		(pts
-			(xy 255.27 130.81) (xy 255.27 135.89)
-		)
-		(stroke
-			(width 0)
-			(type default)
-		)
-	)
-	(wire
-		(pts
 			(xy 68.58 91.44) (xy 91.44 91.44)
 		)
@@
 	(wire
 		(pts
-			(xy 255.27 135.89) (xy 255.27 146.05)
+			(xy 255.27 130.81) (xy 255.27 146.05)
 		)
 		(stroke
@@
 		)
 	)
+	(hierarchical_label "~{RD}"
+		(shape input)
+		(at 251.46 135.89 180)
+		(effects
+			(font
+				(size 1.27 1.27)
+			)
+			(justify right)
+		)
+	)

Commit message: updated parts #s
Parts:
- SW3, SW4, SW5, SW6: MANUFACTURER_PART_NUMBER SH-7070TB -> SH-7070MC
Changed lines of the file:
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@@
 			)
 		)
-		(property "MANUFACTURER_PART_NUMBER" "SH-7070TB"
+		(property "MANUFACTURER_PART_NUMBER" "SH-7070MC"
 			(at 58.42 91.44 0)
 			(hide yes)
@@
 			)
 		)
-		(property "MANUFACTURER_PART_NUMBER" "SH-7070TB"
+		(property "MANUFACTURER_PART_NUMBER" "SH-7070MC"
 			(at 331.47 93.98 0)
 			(hide yes)
@@
 			)
 		)
-		(property "MANUFACTURER_PART_NUMBER" "SH-7070TB"
+		(property "MANUFACTURER_PART_NUMBER" "SH-7070MC"
 			(at 200.66 92.71 0)
 			(hide yes)
@@
 			)
 		)
-		(property "MANUFACTURER_PART_NUMBER" "SH-7070TB"
+		(property "MANUFACTURER_PART_NUMBER" "SH-7070MC"
 			(at 453.39 93.98 0)
 			(hide yes)
