File: Schem/Zephyr-80-IO/IO Controller.kicad_sch (KiCad schematic)
At the start: 44 parts, among them IC1 Z80CTC, IC2 Z80SIO, IC3 Z80SIO, J5 Conn_01x08_Pin, SW1 SW_Push, SW2 SW_Push, U1 74AHCT125, U15 PIC18F57Q84-I/PT, U2 74AHCT1G125, U4 74AHC595, U5 74AHC595, U6 74HC138

Commit message: Fixes to the IO Controller
Connections:
- net GND: no longer U6.5 (~{E1})
- net ~{RD}: now also U6.5 (~{E1})
Changed lines of the file:
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@@
 	)
 	(junction
-		(at 205.74 369.57)
-		(diameter 0)
-		(color 0 0 0 0)
-	)
-	(junction
 		(at 68.58 238.76)
 		(diameter 0)
@@
 	(wire
 		(pts
-			(xy 205.74 369.57) (xy 205.74 381)
-		)
-		(stroke
-			(width 0)
-			(type default)
-		)
-	)
-	(wire
-		(pts
 			(xy 250.19 119.38) (xy 264.16 119.38)
 		)
@@
 	(wire
 		(pts
-			(xy 205.74 369.57) (xy 208.28 369.57)
-		)
-		(stroke
-			(width 0)
-			(type default)
-		)
-	)
-	(wire
-		(pts
 			(xy 134.62 311.15) (xy 144.78 311.15)
 		)
@@
 	(wire
 		(pts
-			(xy 205.74 359.41) (xy 205.74 369.57)
+			(xy 205.74 359.41) (xy 205.74 381)
 		)
 		(stroke
@@
 	(wire
 		(pts
+			(xy 199.39 369.57) (xy 208.28 369.57)
+		)
+		(stroke
+			(width 0)
+			(type default)
+		)
+	)
+	(wire
+		(pts
 			(xy 63.5 213.36) (xy 63.5 215.9)
 		)
@@
 		)
 	)
+	(hierarchical_label "~{RD}"
+		(shape input)
+		(at 199.39 369.57 180)
+		(effects
+			(font
+				(size 1.27 1.27)
+			)
+			(justify right)
+		)
+	)

Commit message: updated parts #s
Parts:
- D1: MANUFACTURER_PART_NUMBER LTST-C150KRKT -> (none)
- IC1: MANUFACTURER_PART_NUMBER 110-44-328-41-001000 -> ICS-628-T
Changed lines of the file:
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@@
 			)
 		)
-		(property "MANUFACTURER_PART_NUMBER" "110-44-328-41-001000"
+		(property "MANUFACTURER_PART_NUMBER" "ICS-628-T"
 			(at 378.46 106.68 0)
 			(hide yes)
@@
 			)
 		)
-		(property "MANUFACTURER_PART_NUMBER" "LTST-C150KRKT"
+		(property "MANUFACTURER_PART_NUMBER" ""
 			(at 62.23 146.05 0)
 			(hide yes)
